File: hardware/DSH-AEGIS.kicad_pcb (KiCad board)
At the start: 2 copper layers, 78 x 101 mm, 15 parts, among them J1 Conn_01x06_Socket, J2 USB_C_Receptacle, SW1 SW_Push, SW2 SW_Push, SW3 SW_Push, SW4 SW_Push, SW5 SW_Push, SW6 SW_Push, U1 ESP32-S3-WROOM-1, U2 ER_OLEDM0.91_1x-I2C, U3 AMS1117-3.3

Commit message: Reorganize repository: move new compact layout into fresh hardware folder
Other:
- board size 78 x 101 mm -> 69.5 x 98.5 mm
